File: hardware/rgb-led-pcb/rgb-led-pcb.kicad_pcb (KiCad board)
At the start: 2 copper layers, 0 parts

Commit message: layout started
Parts:
- added D1: ARGB1313HSTR, local:ARGB1313HSTR, F.Cu at (100.2, 100.0)
- added D2: ARGB1313HSTR, local:ARGB1313HSTR, F.Cu at (110.2, 100.0)
- added D3: ARGB1313HSTR, local:ARGB1313HSTR, F.Cu at (120.2, 100.0)
- added J1: Conn_01x04_MountingPin, local:Molex_Micro_Lock_1x4_Vertical_5055680471, F.Cu at (88.0, 100.0)
- added R1: R, Resistor_SMD:R_1206_3216Metric, F.Cu at (95.2, 100.0)
- added R2: R, Resistor_SMD:R_1206_3216Metric, F.Cu at (105.2, 100.0)
- added R3: R, Resistor_SMD:R_1206_3216Metric, F.Cu at (115.2, 100.0)
Other:
- board outline added: 149.6 x 10.8 mm
